File: Eagle/BackPlane.sch (EAGLE design)
At the start: 34 parts, among them IC2 REG1117, IC4 DS1813, IC5 DS1813, J1 DCJ0202

Commit message: Init
Parts:
- removed IC4: DS1813, ds1813_revised:DS1813SOT-223
- added U$1: DS1233SOT223, TiRoRiN_Libs:DS1233SOT223
- ST1: device TiRoRiN_Libs:IBM8BIT_ISASHORT -> TiRoRiN_Libs:IBM8BIT_ISA
Connections:
- net +5V: now also S3.P, U$1.VCC; no longer IC4.+5V, S3.O
- net GND: now also U$1.GND; no longer IC4.GND
- net N$41: now also ST1CS_7.P; no longer ST1_B10.P
- net N$46: now also ST1CS_6.P; no longer ST1_B15.P
- net N$47: now also ST1CS_5.P; no longer ST1_B16.P
- net N$48: now also ST1CS_4.P; no longer ST1_B17.P
- net N$49: now also ST1CS_3.P; no longer ST1_B18.P
- net N$57: now also ST1CS_2.P; no longer ST1_B26.P
- net N$58: now also ST1CS_1.P; no longer ST1_B27.P
- net N$59: now also ST1CS_0.P; no longer ST1_B28.P
- net RESET: now also U$1.!RESET; no longer IC4./RST
- net VCC: now also S3.O; no longer S3.P
Other:
- moved on the sheet: ST1_+12V, ST1_+3V3, ST1_+5V@1, ST1_+5V@2, ST1_A0, ST1_A1, ST1_A10, ST1_A11, ST1_A12, ST1_A13, ST1_A14, ST1_A15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
