File: Eagle/SBC_65C02_ISA_IRQ_v2.brd (EAGLE design)
At the start: 99.7 x 99.1 mm, 46 parts, among them IC1 74LS00N, IC10 74HC148N, IC11 74HCT574N, IC3 74HCT02N, IC4 DS1813, IC5 DS1813, IC6 74AC00N, IC7 REG1117, IC8 74HCT00N, IC9 74HCT04N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

Commit message: Init
Parts:
- removed C10, C8: 100n, rcl:C050-025X075
- removed C5, C9: (no value), rcl:E3,5-8
- removed IC1: 74LS00N, 74xx-eu:DIL14
- removed IC3: 74HCT02N, 74xx-eu:DIL14
- removed IC6: 74AC00N, 74xx-eu:DIL14
- removed IC7: REG1117, burr-brown:SOT223
- removed IC8: 74HCT00N, 74xx-eu:DIL14
- removed IC9: 74HCT04N, 74xx-eu:DIL14
- removed J1: DCJ0202, con-jack:DCJ0202
- added C11, C12: (no value), rcl:C050-035X075
- added IRQ1_B, NMI_B: (no value), switch-omron:B3F-10XX
- added RN1: (no value), resistor-sil:SIL9
- added SJ1: (no value), jumper:SJ
- ST2: device TiRoRiN_Libs:IBM8BIT -> TiRoRiN_Libs:APP_2X32_SHORT
- moved U$2 81.7 mm to (53.3, 24.8), turned to 270 degrees
- moved R10 76.2 mm to (9.53, 85.7)
- moved R1 75.6 mm to (9.53, 88.3)
- moved R2 74.9 mm to (9.53, 90.8)
- moved R3 74.3 mm to (9.53, 93.3)
- moved C1 31.7 mm to (82.5, 31.8)
- moved R5 17.2 mm to (9.53, 73.0), turned to 180 degrees
- moved R8 14.6 mm to (9.53, 80.6), turned to 0 degrees
- moved IRQ_LED 13.7 mm to (11.4, 59.7), turned to 180 degrees
- moved IO_LED 13.1 mm to (11.4, 66.7), turned to 180 degrees
- moved R7 12.1 mm to (9.53, 75.6), turned to 180 degrees
- moved RESET 11.4 mm to (11.4, 52.7), turned to 180 degrees
- moved C6 10.2 mm to (10.2, 34.3)
- moved S1 10.2 mm to (6.99, 41.3)
- moved QG2 10.2 mm to (10.2, 21.6)
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Connections:
- net N$11 renamed IA1
- net N$18 renamed IA2
- net N$39 renamed BANK_CS
- net N$9 renamed IA0
- removed net IO_CS_N: IC1.10, IC1.12, IC8.10, IC9.12
- removed net N$1: IC8.4, IC9.2
- removed net N$10: IC1.5, IC9.10
- removed net N$12: C10.2, C8.2, C9.-, IC7.1
- removed net N$14: IC3.3, IC8.6
- removed net N$15: IC3.1, IC9.5
- removed net N$16: IC3.4, IC3.9
- removed net N$17: IC3.10, IC9.9
- removed net N$19: U$2.1
- removed net N$20: U$2.2
- removed net N$21: U$2.3
- removed net N$22: U$2.4
- removed net N$23: U$2.5
- removed net N$24: U$2.6
- removed net N$26: U$2.7
- removed net N$27: U$2.8
- removed net N$28: U$2.9
- removed net N$29: U$2.10
- removed net N$3: IC3.11, IC6.6
- removed net N$32: U$2.12
- removed net N$33: U$2.24
- removed net N$34: U$2.23
- removed net N$35: U$2.22
- removed net N$36: U$2.21
- removed net N$37: U$2.20
- removed net N$38: U$2.19
- removed net N$4: IC3.12, IC6.3
- removed net N$42: U$2.17
- removed net N$43: U$2.16
- removed net N$44: U$2.15
- removed net N$45: U$2.14
- removed net N$5: IC8.5, IC9.4
- removed net N$7: IC3.2, IC3.8, IC8.3
- removed net N$8: IC3.13, IC8.9
- new net CS_0: ST2.B28
- new net CS_1: ST2.B27
- new net CS_2: ST2.B26
- new net CS_3: ST2.B18
- new net CS_4: ST2.B17
- new net CS_5: ST2.B16
- new net CS_6: ST2.B15
- new net CS_7: ST2.B10
- new net DTR: JP3.1, SJ1.2
- new net RAM_CS: IC2.20, U$2.22
- net +3V3: no longer C8.1, C9.+, IC7.2
- net +5V: now also C11.1, C12.1, JP3.4, RN1.1, U$2.24; no longer C10.1, C5.+, IC1.14, IC3.14, IC6.14, IC7.3, IC8.14, IC9.14, J1.1
- net A10: now also U$2.7; no longer IC6.5
- net A11: now also U$2.6; no longer IC6.4
- net A12: now also U$2.5; no longer IC3.6, IC9.3
- net A13: now also U$2.4; no longer IC3.5, IC9.1
- net A14: now also U$2.3; no longer IC8.2
- net A15: now also U$2.2; no longer IC2.20, IC8.1
- net A8: now also U$2.9; no longer IC6.2
- net A9: now also U$2.8; no longer IC6.1
- net ACIA_CS: now also U$2.20; no longer IC8.8
- net GND: now also C11.2, C12.2, IRQ1_B.1, NMI_B.1, U$2.12; no longer C5.-, IC1.7, IC3.7, IC6.7, IC8.7, IC9.7, J1.2, J1.3
- net IOR: now also U$2.15; no longer IC1.8
- net IOW: now also U$2.14; no longer IC1.11
- net IO_CS: now also U$2.21; no longer IC9.13, IC9.6
- net IRQ0: now also RN1.2
- net IRQ1: now also IRQ1_B.3, RN1.3
- net IRQ2: now also RN1.4
- net IRQ3: now also RN1.5
- net IRQ4: now also RN1.6
- net IRQ5: now also RN1.7
- net IRQ6: now also RN1.8
- net IRQ7: now also RN1.9
- net IRQ_CS: now also U$2.19
- net MEMR: now also U$2.17; no longer IC1.13, IC1.3
- net MEMW: now also U$2.16; no longer IC1.6, IC1.9
- net NMI: now also NMI_B.3
- net PHI2: now also U$2.1; no longer IC1.2, IC1.4
- net RESET: now also SJ1.1
- net ROM_CS: now also U$2.23; no longer IC9.8
- net RW: now also U$2.10; no longer IC1.1, IC9.11
Routing:
- net GND: track 0.00 -> 485.4 mm, vias 0 -> 9
- net +5V: track 0.00 -> 462.5 mm, vias 0 -> 7
- net RESET: track 0.00 -> 277.0 mm, vias 0 -> 8
- net PHI2: track 0.00 -> 229.8 mm, vias 0 -> 6
- net RW: track 0.00 -> 221.8 mm, vias 0 -> 3
- net IRQ: track 0.00 -> 187.5 mm, vias 0 -> 1
- net D3: track 0.00 -> 177.3 mm, vias 0 -> 7
- net D7: track 0.00 -> 177.1 mm, vias 0 -> 4
- net D5: track 0.00 -> 161.5 mm, vias 0 -> 6
- net NMI: track 0.00 -> 160.9 mm, vias 0 -> 2
- net IRQ1: track 0.00 -> 157.5 mm, vias 0 -> 4
- net A8: track 0.00 -> 155.7 mm, vias 0 -> 3
- net D1: track 0.00 -> 155.4 mm, vias 0 -> 3
- net D6: track 0.00 -> 155.4 mm, vias 0 -> 6
- net D4: track 0.00 -> 153.8 mm, vias 0 -> 4
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- added copper zone on layer 1, net GND
- added copper zone on layer 16, net GND
Other:
- board text added: "+5v"
- board text added: "22pF"
- board text added: "DTR"
- board text added: "DTR = RST"
- board text added: "IO"
- board text added: "IRQ"
- board text added: "IRQ7"
- board text added: "NMI"
- board text added: "RST"
- board text removed: "5VDC IN"
- board text removed: "74xx00"
