File: Eagle/SBC_65C02_ISA_IRQ_v2.sch (EAGLE design)
At the start: 41 parts, among them IC10 74HC148N, IC11 74HCT574N, IC4 DS1813, IC5 DS1813, Q1 1,8432MHz, U1 W65C02SP

Commit message: Init
Parts:
- ST2: device TiRoRiN_Libs:IBM8BIT_ISA -> TiRoRiN_Libs:IBM8BIT_ISASHORT
Connections:
- new net CS_0: ST2CS_0.P
- new net CS_1: ST2CS_1.P
- new net CS_2: ST2CS_2.P
- new net CS_3: ST2CS_3.P
- new net CS_4: ST2CS_4.P
- new net CS_5: ST2CS_5.P
- new net CS_6: ST2CS_6.P
- new net CS_7: ST2CS_7.P
Other:
- moved on the sheet: R9
Changed lines of the file:
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@@
 <part name="R9" library="rcl" library_urn="urn:adsk.eagle:library:334" deviceset="R-EU_" device="0207/10" package3d_urn="urn:adsk.eagle:package:23491/2" value="22k"/>
 <part name="JP3" library="pinhead" library_urn="urn:adsk.eagle:library:325" deviceset="PINHD-1X6" device="/90" package3d_urn="urn:adsk.eagle:package:22475/2"/>
-<part name="ST2" library="TiRoRiN_Libs" deviceset="IBM8BIT_ISA" device="" package3d_urn="urn:adsk.eagle:package:9255/1"/>
+<part name="ST2" library="TiRoRiN_Libs" deviceset="IBM8BIT_ISA" device="SHORT" package3d_urn="urn:adsk.eagle:package:9255/1"/>
 <part name="IRQ_LED" library="led" library_urn="urn:adsk.eagle:library:259" deviceset="LED" device="5MM" package3d_urn="urn:adsk.eagle:package:15799/2"/>
 <part name="R6" library="resistor" library_urn="urn:adsk.eagle:library:348" deviceset="R-EU_" device="0207/10" package3d_urn="urn:adsk.eagle:package:23491/2" value="680R"/>
@@
 <part name="ROM_1" library="jump-0r-smd" library_urn="urn:adsk.eagle:library:251" deviceset="0R-JUMP" device="A" package3d_urn="urn:adsk.eagle:package:15385/1"/>
 <part name="ROM_27" library="jump-0r-smd" library_urn="urn:adsk.eagle:library:251" deviceset="0R-JUMP" device="A" package3d_urn="urn:adsk.eagle:package:15385/1"/>
-<part name="IC10" library="74xx-eu" library_urn="urn:adsk.eagle:library:85" deviceset="74*148" device="N" package3d_urn="urn:adsk.eagle:package:2009/1" technology="HC"/>
-<part name="IC11" library="74xx-eu" library_urn="urn:adsk.eagle:library:85" deviceset="74*574" device="N" package3d_urn="urn:adsk.eagle:package:2017/1" technology="HCT"/>
+<part name="IC10" library="74xx-eu" library_urn="urn:adsk.eagle:library:85" deviceset="74*148" device="N" package3d_urn="urn:adsk.eagle:package:922/2" technology="HC"/>
+<part name="IC11" library="74xx-eu" library_urn="urn:adsk.eagle:library:85" deviceset="74*574" device="N" package3d_urn="urn:adsk.eagle:package:16429/2" technology="HCT"/>
 <part name="U$2" library="TiRoRiN_Libs" deviceset="GAL22V10" device=""/>
 <part name="RN1" library="resistor-sil" library_urn="urn:adsk.eagle:library:347" deviceset="G08R" device="" package3d_urn="urn:adsk.eagle:package:25282/1"/>
@@
 <attribute name="VALUE" x="-173.101" y="24.384" size="1.778" layer="96" rot="R90"/>
 </instance>
-<instance part="R9" gate="G$1" x="-127" y="-25.4" smashed="yes" rot="R90">
-<attribute name="NAME" x="-128.4986" y="-29.21" size="1.778" layer="95" rot="R90"/>
-<attribute name="VALUE" x="-128.778" y="-24.13" size="1.778" layer="96" rot="R90"/>
+<instance part="R9" gate="G$1" x="-124.46" y="-25.4" smashed="yes" rot="R90">
+<attribute name="NAME" x="-125.9586" y="-29.21" size="1.778" layer="95" rot="R90"/>
+<attribute name="VALUE" x="-126.238" y="-24.13" size="1.778" layer="96" rot="R90"/>
 </instance>
 <instance part="JP3" gate="A" x="-177.8" y="-5.08" smashed="yes" rot="R180">
@@
 <attribute name="NAME" x="-135.255" y="49.8348" size="1.778" layer="95"/>
 </instance>
-<instance part="ST2" gate="_B10" x="-139.7" y="53.34" smashed="yes">
+<instance part="ST2" gate="CS_7" x="-139.7" y="53.34" smashed="yes">
 <attribute name="NAME" x="-135.255" y="52.3748" size="1.778" layer="95"/>
 </instance>
@@
 <attribute name="NAME" x="-135.255" y="62.5348" size="1.778" layer="95"/>
 </instance>
-<instance part="ST2" gate="_B15" x="-139.7" y="66.04" smashed="yes">
+<instance part="ST2" gate="CS_6" x="-139.7" y="66.04" smashed="yes">
 <attribute name="NAME" x="-135.255" y="65.0748" size="1.778" layer="95"/>
 </instance>
-<instance part="ST2" gate="_B16" x="-139.7" y="68.58" smashed="yes">
+<instance part="ST2" gate="CS_5" x="-139.7" y="68.58" smashed="yes">
 <attribute name="NAME" x="-135.255" y="67.6148" size="1.778" layer="95"/>
 </instance>
-<instance part="ST2" gate="_B17" x="-139.7" y="71.12" smashed="yes">
+<instance part="ST2" gate="CS_4" x="-139.7" y="71.12" smashed="yes">
 <attribute name="NAME" x="-135.255" y="70.1548" size="1.778" layer="95"/>
 </instance>
-<instance part="ST2" gate="_B18" x="-139.7" y="73.66" smashed="yes">
+<instance part="ST2" gate="CS_3" x="-139.7" y="73.66" smashed="yes">
 <attribute name="NAME" x="-135.255" y="72.6948" size="1.778" layer="95"/>
 </instance>
@@
 <attribute name="NAME" x="-135.255" y="90.4748" size="1.778" layer="95"/>
 </instance>
-<instance part="ST2" gate="_B26" x="-139.7" y="93.98" smashed="yes">
+<instance part="ST2" gate="CS_2" x="-139.7" y="93.98" smashed="yes">
 <attribute name="NAME" x="-135.255" y="93.0148" size="1.778" layer="95"/>
 </instance>
-<instance part="ST2" gate="_B27" x="-139.7" y="96.52" smashed="yes">
+<instance part="ST2" gate="CS_1" x="-139.7" y="96.52" smashed="yes">
 <attribute name="NAME" x="-135.255" y="95.5548" size="1.778" layer="95"/>
 </instance>
-<instance part="ST2" gate="_B28" x="-139.7" y="99.06" smashed="yes">
+<instance part="ST2" gate="CS_0" x="-139.7" y="99.06" smashed="yes">
 <attribute name="NAME" x="-135.255" y="98.0948" size="1.778" layer="95"/>
 </instance>
@@
 </instances>
 <busses>
-<bus name="A8,A9,A10,A11,ACIA_CS,IO_CS,IO_CS_N,N$3,N$4,N$8,N$10">
+<bus name="A8,A9,A10,A11,ACIA_CS,IO_CS,IO_CS_N,N$3,N$10">
 <segment>
 <wire x1="-195.58" y1="27.94" x2="-111.76" y2="27.94" width="0.762" layer="92"/>
@@
 </segment>
 <segment>
-<wire x1="-127" y1="-20.32" x2="-127" y2="-17.78" width="0.1524" layer="91"/>
+<wire x1="-124.46" y1="-20.32" x2="-124.46" y2="-17.78" width="0.1524" layer="91"/>
 <pinref part="R9" gate="G$1" pin="2"/>
 <label x="-127" y="-20.32" size="1.778" layer="95"/>
@@
 <segment>
 <pinref part="U$4" gate="G$1" pin="CS0"/>
-<wire x1="-139.7" y1="-30.48" x2="-127" y2="-30.48" width="0.1524" layer="91"/>
+<wire x1="-139.7" y1="-30.48" x2="-124.46" y2="-30.48" width="0.1524" layer="91"/>
 <pinref part="R9" gate="G$1" pin="1"/>
 <label x="-139.7" y="-30.48" size="1.778" layer="95"/>
@@
 </segment>
 </net>
+<net name="CS_0" class="0">
+<segment>
+<pinref part="ST2" gate="CS_0" pin="P"/>
+<wire x1="-142.24" y1="99.06" x2="-149.86" y2="99.06" width="0.1524" layer="91"/>
+<label x="-149.86" y="99.06" size="1.778" layer="95"/>
+</segment>
+</net>
+<net name="CS_1" class="0">
+<segment>
+<pinref part="ST2" gate="CS_1" pin="P"/>
+<wire x1="-142.24" y1="96.52" x2="-149.86" y2="96.52" width="0.1524" layer="91"/>
+<label x="-149.86" y="96.52" size="1.778" layer="95"/>
+</segment>
+</net>
+<net name="CS_2" class="0">
+<segment>
+<pinref part="ST2" gate="CS_2" pin="P"/>
+<wire x1="-142.24" y1="93.98" x2="-149.86" y2="93.98" width="0.1524" layer="91"/>
+<label x="-149.86" y="93.98" size="1.778" layer="95"/>
+</segment>
+</net>
+<net name="CS_3" class="0">
+<segment>
+<pinref part="ST2" gate="CS_3" pin="P"/>
+<wire x1="-142.24" y1="73.66" x2="-149.86" y2="73.66" width="0.1524" layer="91"/>
+<label x="-149.86" y="73.66" size="1.778" layer="95"/>
+</segment>
+</net>
+<net name="CS_4" class="0">
+<segment>
+<pinref part="ST2" gate="CS_4" pin="P"/>
+<wire x1="-142.24" y1="71.12" x2="-149.86" y2="71.12" width="0.1524" layer="91"/>
+<label x="-149.86" y="71.12" size="1.778" layer="95"/>
+</segment>
+</net>
+<net name="CS_5" class="0">
+<segment>
+<pinref part="ST2" gate="CS_5" pin="P"/>
+<wire x1="-142.24" y1="68.58" x2="-149.86" y2="68.58" width="0.1524" layer="91"/>
+<label x="-149.86" y="68.58" size="1.778" layer="95"/>
+</segment>
+</net>
+<net name="CS_6" class="0">
+<segment>
+<pinref part="ST2" gate="CS_6" pin="P"/>
+<wire x1="-142.24" y1="66.04" x2="-149.86" y2="66.04" width="0.1524" layer="91"/>
+<label x="-149.86" y="66.04" size="1.778" layer="95"/>
+</segment>
+</net>
+<net name="CS_7" class="0">
+<segment>
+<pinref part="ST2" gate="CS_7" pin="P"/>
+<wire x1="-142.24" y1="53.34" x2="-152.4" y2="53.34" width="0.1524" layer="91"/>
+<label x="-149.86" y="53.34" size="1.778" layer="95"/>
+</segment>
+</net>
