File: Eagle/SBC_TMS9918A_ISA.brd (EAGLE design)
At the start: 99.7 x 99.1 mm, 33 parts, among them IC2 74HCT85N, IC3 TMS9918, IC4 74HCT32N, IC5 74HCT04N, IC6 74HCT574N, IC7 74HCT574N, IC8 74HCT574N, Q2 BC337, X1 736880-49

Commit message: Init
Connections:
- removed net !CS: IC4.8
- net CS: now also IC4.8
Routing:
- net IOR: track 74.7 -> 163.6 mm, vias 3 -> 4
- net !OE: track 90.0 -> 152.8 mm, vias 2 -> 3
- net VA4: track 50.0 -> 98.1 mm, vias 2 -> 1
- net VA1: track 31.6 -> 73.0 mm, vias 0 -> 3
- net VA0: track 39.9 -> 80.9 mm, vias 1 -> 3
- net R/!W: track 106.3 -> 140.8 mm, vias 1 -> 3
- net +5V: track 288.2 -> 321.3 mm
- net VA6: track 47.5 -> 80.5 mm, vias 1 -> 0
- net CS: track 9.00 -> 39.4 mm, vias 0 -> 4
- net GND: track 321.6 -> 347.0 mm, vias 0 -> 1
- net VD3: track 69.8 -> 94.6 mm, vias 2 -> 3
- net VD1: track 62.3 -> 82.7 mm
- net A10_S: track 31.8 -> 52.0 mm
- net VD6: track 103.4 -> 84.2 mm, vias 1 -> 3
- net A0: track 63.4 -> 81.2 mm, vias 2 -> 1
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Other:
- board text added: "TMS9918A V1"
