File: Eagle/SBC_TMS9918A_ISA.sch (EAGLE design)
At the start: 33 parts, among them IC2 74HCT85N, IC3 TMS9918, IC4 74HCT32N, IC5 74HCT04N, IC6 74HCT574N, IC7 74HCT574N, IC8 74HCT574N, Q2 BC337, X1 736880-49

Commit message: Init
Connections:
- removed net !CS: IC4C.O
- net CS: now also IC4C.O
Changed lines of the file:
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@@
 </variantdefs>
 <classes>
-<class number="0" name="default" width="0.1524" drill="0.2">
-<clearance class="0" value="0.1524"/>
+<class number="0" name="default" width="0.381" drill="0.2">
+<clearance class="0" value="0.254"/>
 </class>
 <class number="1" name="power" width="0.508" drill="0.6604">
@@
 <clearance class="1" value="0.254"/>
 </class>
-<class number="2" name="data" width="0.254" drill="0.6604">
+<class number="2" name="data" width="0.381" drill="0.6604">
 <clearance class="0" value="0.254"/>
 <clearance class="1" value="0.254"/>
@@
 </segment>
 </net>
-<net name="!CS" class="0">
-<segment>
-<pinref part="IC4" gate="C" pin="O"/>
-<wire x1="-68.58" y1="152.4" x2="-50.8" y2="152.4" width="0.1524" layer="91"/>
-<label x="-55.88" y="152.4" size="1.778" layer="95"/>
-</segment>
-</net>
 <net name="!RAS" class="0">
 <segment>
@@
 <label x="-33.02" y="193.04" size="1.778" layer="95"/>
 </segment>
-</net>
+<segment>
+<pinref part="IC4" gate="C" pin="O"/>
+<wire x1="-68.58" y1="152.4" x2="-50.8" y2="152.4" width="0.1524" layer="91"/>
+<label x="-55.88" y="152.4" size="1.778" layer="95"/>
+</segment>
+</net>
