File: Eagle/SBC_65C02_IRQ_BigBoard_v10-2-1.sch (EAGLE design)
At the start: 114 parts, among them IC1 REG1117_3V3, IC10 74AC00N, IC11 74HCT139N, IC12 74AC00N, IC14 ATTINY26-16PU, IC17 74HC148N, IC19 R6551, IC2 74HC74N, IC20 SAA, IC21 74AC32N, IC3 74HC74N, IC4 W65C02SP, IC5 28C64AP, IC6 62256, IC7 62256, IC8 DS1233, IC9 74HCT139N, J1 DCJ0202, J2 AVR_SPI_PROG_3X2NS, Q1 1,8432MHz, X5 PG203J

Commit message: Add new schematic for SBC 65C02 IRQ BigBoard v10-2-1
Parts:
- removed C31: (no value), rcl:C-EU050-025X075
- removed C32, C33, C34, C35: 10n, rcl:C-EU050-025X075
- removed C36, C37: 100n, rcl:C-EU050-025X075
- removed IC20: SAA, TiRoRiN_Libs:SAA1099DIL18
- removed L1: (no value), rcl:L-EU0207/10
- removed R18, R19: 22k, rcl:R-EU_0207/10
- removed R20, R21, R22, R23: 1k, rcl:R-EU_0207/10
- removed X5: PG203J, con-hirschmann:PG203J
- added C16, C18: (no value), rcl:C-EU050-025X075
- added IC27: 74HC574N, 74xx-eu:74HC574N
- added J4: (no value), SparkFun-Connectors:USB_C2-LAYER
- added SJ3, SJ4: (no value), jumper:SJ
- added U$1: MCP2221A-I/P, MCP2221:MCP2221A-I/P
- IC16: value (none) -> VIA1
- IC18: value (none) -> VIA2
- JP6: device pinhead:PINHD-1X11 -> pinhead:PINHD-2X12
Connections:
- net !D_CS renamed !$DXXX_CS
- net !SPI_CS renamed !VERA_CS
- removed net !RAM_CS: JP6.7
- removed net N$1: L1.2, R18.2, R19.2
- removed net N$15: C34.2, C36.1, R22.2
- removed net N$16: C35.2, C37.1, R23.2
- removed net OUTL: C32.2, IC20.OUTL, R20.2, R22.1
- removed net OUTR: C33.2, IC20.OUTR, R21.2, R23.1
- removed net RESET: IC16VIA.!RESB, IC18VIA.!RESB, IC19.RES, IC4.RESB, IC8.!RESET, LED5.C, R13.2, S3.P, S3.P1, SJ1.1, X1-B2.P, X2-B2.P, X3-B2.P
- removed net SAA_DACK: IC20.DTACK, R18.1
- removed net SAA_IREF: IC20.IREF, R19.1
- removed net SOUND_L: C36.2, X5.2
- removed net SOUND_R: C37.2, X5.5
- new net !$C4-7: IC21B.I0, IC21C.I0, IC9A.Y1
- new net !IRQ_CS: IC21C.O, IC27A.OC
- new net !RESET: IC16VIA.!RESB, IC18VIA.!RESB, IC19.RES, IC4.RESB, IC8.!RESET, JP6.12, LED5.C, R13.2, S3.P, S3.P1, SJ1.1, SJ3.1, SJ4.2, X1-B2.P, X2-B2.P, X3-B2.P
- new net !USB_RESET: SJ4.1, U$1.!RST
- new net D+: J4.D+, U$1.USB+
- new net D-: J4.D-, U$1.USB-
- new net N$36: JP6.23
- new net N$39: IC17A.A0, IC27A.2D
- new net N$40: IC17A.A1, IC27A.3D
- new net N$41: IC17A.A2, IC27A.4D
- new net N$45: J4.CC1
- new net N$52: JP6.24
- net !A7: now also IC21C.I1
- net !AA_CS: now also IC21B.O; no longer IC9A.Y1, JP6.10
- net !AA_CS_WR: no longer IC20.!CS, IC20.!WR
- net !ACIA_CS: no longer JP6.8
- net !HRAM_CS: no longer JP6.6
- net !IO_CS: no longer JP6.5
- net !MEMR: now also JP6.16; no longer JP6.3
- net !MEMW: now also JP6.13; no longer JP6.2
- net !ROM_CS: no longer JP6.4
- net !VIA_CS: no longer JP6.9
- net +5V: now also C16.1, C18.1, IC27P.VCC, J4.VBUS, JP6.1, U$1.VDD, U$1.VUSB; no longer C31.2, IC20.+5V, L1.1, R20.1, R21.1
- net 8MHZ: no longer IC20.CLK
- net A0: now also JP6.19; no longer IC20.A0
- net A1: now also JP6.20
- net A2: now also JP6.17
- net A3: now also JP6.18
- net A4: now also JP6.15
- net A7: now also IC21B.I1
- net AVR_RST: now also SJ3.2
- net D0: now also IC27A.1Q, JP6.10; no longer IC20.D0
- net D1: now also IC27A.2Q, JP6.9; no longer IC20.D1
- net D2: now also IC27A.3Q, JP6.8; no longer IC20.D2
- net D3: now also IC27A.4Q, JP6.7; no longer IC20.D3
- net D4: now also IC27A.5Q, JP6.6; no longer IC20.D4
- net D5: now also IC27A.6Q, JP6.5; no longer IC20.D5
- net D6: now also IC27A.7Q, JP6.4; no longer IC20.D6
- net D7: now also IC27A.8Q, JP6.3; no longer IC20.D7
- net GND: now also C16.2, C18.2, IC27A.1D, IC27A.5D, IC27A.6D, IC27A.7D, IC27A.8D, IC27P.GND, J4.GND, J4.SHLD, JP6.2, JP6.21, JP6.22, U$1.GND; no longer C31.1, C32.1, C33.1, C34.1, C35.1, IC20.GND, JP6.1, X5.1
- net IRQ2: now also JP6.14
- net PHI2: now also IC27A.CLK
- net RX: now also U$1.URX
- net TX: now also U$1.UTX
Other:
- note added: "HEX OUT C0-3XX !TMS_CS C4-7XX !C4-7 C40-7X !AA_CS C48-F0 !IRQ_CS C8-BXX !ACIA_CS CCXX !VIA_CS CC0-7X !VIA2_CS CC8-FX !VIA1_CS CDXX !DEV0 CEXX !DEV1 CFXX !DEV2"
- note removed: "HEX OUT C0-3XX !SPI_CS C4-7XX !AA_CS C8-BXX !ACIA_CS CCXX !VIA_CS CC0-7X !VIA1_CS CC8-FX !VIA1_CS CDXX !DEV0 CEXX !DEV1 CFXX !DEV2"
